File: PCB/R3M1XXX.kicad_sch (KiCad schematic)
At the start: 0 parts

Commit message: schematic wip
Parts:
- added A1: Raspberry_Pi_Pico_THT, PCM_SL_Development_Boards:raspberry_pi_pico_THT, symbol PCM_SL_Development_Board:Raspberry_Pi_Pico_THT
Changed lines of the file:
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@@
 	(generator_version "8.0")
 	(paper "A4")
+	(symbol
+		(lib_id "PCM_SL_Development_Board:Raspberry_Pi_Pico_THT")
+		(at 77.47 80.01 0)
+		(unit 1)
+		(exclude_from_sim no)
+		(in_bom yes)
+		(on_board yes)
+		(dnp no)
+		(fields_autoplaced yes)
+		(property "Reference" "A1"
+			(at 88.5541 45.72 0)
+			(effects
+				(font
+					(size 1.27 1.27)
+				)
+				(justify left)
+			)
+		)
+		(property "Value" "Raspberry_Pi_Pico_THT"
+			(at 88.5541 48.26 0)
+			(effects
+				(font
+					(size 1.27 1.27)
+				)
+				(justify left)
+			)
+		)
+		(property "Footprint" "PCM_SL_Development_Boards:raspberry_pi_pico_THT"
+			(at 77.47 106.68 0)
+			(effects
+				(font
+					(size 1.27 1.27)
+				)
+				(hide yes)
+			)
+		)
+		(property "Datasheet" ""
+			(at 77.47 68.58 0)
+			(effects
+				(font
+					(size 1.27 1.27)
+				)
+				(hide yes)
+			)
+		)
+		(property "Description" "Development Board with RP2040 MCU "
+			(at 77.47 80.01 0)
+			(effects
+				(font
+					(size 1.27 1.27)
+				)
+				(hide yes)
+			)
+		)
+		(pin "26"
+		)
+		(pin "27"
+		)
+		(pin "12"
+		)
+		(pin "13"
+		)
+		(pin "19"
+		)
+		(pin "31"
+		)
+		(pin "32"
+		)
+		(pin "1"
+		)
+		(pin "2"
+		)
+		(pin "33"
+		)
+		(pin "34"
+		)
+		(pin "35"
+		)
+		(pin "36"
+		)
+		(pin "20"
+		)
+		(pin "21"
+		)
+		(pin "22"
+		)
+		(pin "23"
+		)
+		(pin "10"
+		)
+		(pin "3"
+		)
+		(pin "30"
+		)
+		(pin "6"
+		)
+		(pin "7"
+		)
+		(pin "39"
+		)
+		(pin "4"
+		)
+		(pin "16"
+		)
+		(pin "18"
+		)
+		(pin "40"
+		)
+		(pin "5"
+		)
+		(pin "28"
+		)
+		(pin "29"
+		)
+		(pin "8"
+		)
+		(pin "9"
+		)
+		(pin "17"
+		)
+		(pin "11"
+		)
+		(pin "15"
+		)
+		(pin "24"
+		)
+		(pin "25"
+		)
+		(pin "37"
+		)
+		(pin "38"
+		)
+		(pin "14"
+		)
+		(instances
+			(project ""
+				(path "/734751e6-bef2-4814-98c0-5802ec8506b2"
+					(reference "A1")
+					(unit 1)
+				)
+			)
+		)
+	)
 	(sheet
 		(at 238.76 69.85)
