File: PCB/encoders.kicad_sch (KiCad schematic)
At the start: 34 parts, among them SW1 RotaryEncoder_Switch, SW13 SW, SW14 SW, SW2 RotaryEncoder_Switch, SW3 RotaryEncoder_Switch, SW4 RotaryEncoder_Switch

Commit message: schematic wip
Parts:
- added U1, U2: SSD1357, symbol r3m1xxx_Library:SSD1357-OLED
- added U3: CD74HC4067M, Package_SO:SOIC-24W_7.5x15.4mm_P1.27mm, symbol 74xx:CD74HC4067M
Connections:
- net +5V: now also U1.1 (VCC), U2.1 (VCC), U3.24 (VCC)
- net FNSW: now also U3.8 (I1)
- net GND: now also U1.2 (GND), U2.2 (GND), U3.12 (GND), U3.15 (~{E})
- net ROT-1A: now also U3.3 (I6)
- net ROT-1B: now also U3.2 (I7)
- net ROT-1SW: now also U3.7 (I2)
- net ROT-2A: now also U3.23 (I8)
- net ROT-2B: now also U3.22 (I9)
- net ROT-2SW: now also U3.6 (I3)
- net ROT-3A: now also U3.21 (I10); no longer C8.1, R8.2, SW3.A
- net ROT-3B: now also U3.20 (I11); no longer C7.1, R7.2, SW3.B
- net ROT-3SW: now also U3.5 (I4)
- net ROT-4A: now also U3.19 (I12)
- net ROT-4B: now also U3.18 (I13)
- net ROT-4SW: now also U3.4 (I5)
- net SFTSW: now also U3.9 (I0)
- new net: C7.1, R7.2, SW3.B
- new net: C8.1, R8.2, SW3.A
- new net MPLEX-B: U3.1 (COM)
- new net MPLEX-S0: U3.10 (S0)
- new net MPLEX-S1: U3.11 (S1)
- new net MPLEX-S2: U3.14 (S2)
- new net MPLEX-S3: U3.13 (S3)
- new net SLCK: U1.4 (CLK), U2.4 (CLK)
- no-connect marks 0 -> 2
Other:
- moved on the sheet: C1, C10, C11, C12, C2, C21, C22, C3, C4, C5, C6, C7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

Commit message: wip
Parts:
- removed U2: SSD1357, symbol r3m1xxx_Library:SSD1357-OLED
- added D1, D2: WS2812B, LED_SMD:LED_WS2812B_PLCC4_5.0x5.0mm_P3.2mm, symbol LED:WS2812B
- added J1, J2, J3: Conn_01x06, symbol Connector_Generic:Conn_01x06
- added J4: Conn_01x04, symbol Connector_Generic:Conn_01x04
- added U2: ST7789, symbol r3m1xxx_Library:ST7789-oled
- U1: value SSD1357 -> ST7789; symbol r3m1xxx_Library:SSD1357-OLED -> r3m1xxx_Library:ST7789-oled
Connections:
- net +5V: now also D1.1 (VDD), D2.1 (VDD), J4.2 (Pin_2); no longer U1.1 (VCC)
- net GND: now also U1.1 (GND), D1.3 (VSS), D2.3 (VSS), J1.1 (Pin_1), J2.1 (Pin_1), J3.1 (Pin_1), J4.1 (Pin_1), U2.1 (GND); no longer U1.2 (GND)
- net MPLEX-B: now also J1.2 (Pin_2)
- net MPLEX-S0: now also J1.3 (Pin_3)
- net MPLEX-S1: now also J1.4 (Pin_4)
- net MPLEX-S2: now also J1.5 (Pin_5)
- net MPLEX-S3: now also J1.6 (Pin_6)
- net SPI0_SCK: now reaches U1.3 (SCL)
- net SPI0_SCK: now also U1.7 (CS), J2.3 (Pin_3)
- net SPI0_RX: now reaches U1.5 (RES)
- net SPI0_RX: now also J2.5 (Pin_5)
- net SPI0_CS: now reaches U1.6 (DC)
- net SPI0_CS: now also J2.6 (Pin_6)
- net SLCK renamed SPI0_TX
- net SPI0_TX: now also J2.4 (Pin_4)
- new net: D1.2 (DOUT), D2.4 (DIN)
- new net 3V3: J2.2 (Pin_2), J3.2 (Pin_2), U1.2 (VCC), U1.8 (BLK), U2.2 (VCC), U2.8 (BLK)
- new net NP2IN: D1.4 (DIN), J4.3 (Pin_3)
- new net NP2OUT: D2.2 (DOUT), J4.4 (Pin_4)
- new net SPI1_CS: J3.6 (Pin_6), U2.6 (DC)
- new net SPI1_RX: J3.5 (Pin_5), U2.5 (RES)
- new net SPI1_SCK: J3.3 (Pin_3), U2.3 (SCL), U2.7 (CS)
- new net SPI1_TX: J3.4 (Pin_4), U2.4 (SDA)
Other:
- moved on the sheet: U3
