File: PCB/fx.kicad_sch (KiCad schematic)
At the start: 32 parts, among them SW10 SW, SW11 SW, SW12 SW, SW5 SW, SW6 SW, SW7 SW, SW8 SW, SW9 SW

Commit message: wip
Parts:
- added D10, D3, D4, D5, D6, D7, D8, D9: WS2812B, LED_SMD:LED_WS2812B_PLCC4_5.0x5.0mm_P3.2mm, symbol LED:WS2812B
Connections:
- net +5V: now also D10.1 (VDD), D3.1 (VDD), D4.1 (VDD), D5.1 (VDD), D6.1 (VDD), D7.1 (VDD), D8.1 (VDD), D9.1 (VDD)
- net GND: now also D10.3 (VSS), D3.3 (VSS), D4.3 (VSS), D5.3 (VSS), D6.3 (VSS), D7.3 (VSS), D8.3 (VSS), D9.3 (VSS)
- net POT1: now reaches RV1.2
- net POT6: now reaches RV6.2
- net POT5: now reaches RV5.2
- net POT7: now reaches RV7.2
- net POT2: now reaches RV2.2
- net POT3: now reaches RV3.2
- new net: D6.2 (DOUT), D7.4 (DIN)
- new net: D5.2 (DOUT), D6.4 (DIN)
- new net: D7.2 (DOUT), D8.4 (DIN)
- new net: D4.2 (DOUT), D5.4 (DIN)
- new net: D3.2 (DOUT), D4.4 (DIN)
- new net: D10.4 (DIN), D9.2 (DOUT)
- new net: D8.2 (DOUT), D9.4 (DIN)
- new net NP1IN: D3.4 (DIN)
- new net NP1OUT: D10.2 (DOUT)
Other:
- moved on the sheet: RV1, RV2, RV3, RV4, RV5, RV6, RV7, RV8
