File: KiCAD/X01/encoders.kicad_sch (KiCad schematic)
At the start: 43 parts, among them J1 Conn_01x06, J2 Conn_01x06, J3 Conn_01x06, J4 Conn_01x04, SW1 RotaryEncoder_Switch, SW13 SW, SW14 SW, SW2 RotaryEncoder_Switch, SW3 RotaryEncoder_Switch, SW4 RotaryEncoder_Switch, U1 ST7789, U2 ST7789, U3 CD74HC4067M

Commit message: M01 & X01
Parts:
- J1: value Conn_01x06 -> Conn_B1
- J2: value Conn_01x06 -> Conn_B3
- J3: value Conn_01x06 -> Conn_B4
- J4: value Conn_01x04 -> Conn_B2
Changed lines of the file:
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@@
 		)
 		(instances
-			(project ""
+			(project "R3M1XXX"
 				(path "/734751e6-bef2-4814-98c0-5802ec8506b2/1f2cf491-dbdb-4a6a-9515-9e3b3af8ab6f"
 					(reference "U1")
@@
 			)
 		)
-		(property "Value" "Conn_01x06"
+		(property "Value" "Conn_B3"
 			(at 160.02 133.3499 0)
 			(effects
@@
 			)
 		)
-		(property "Value" "Conn_01x06"
+		(property "Value" "Conn_B1"
 			(at 127 134.6199 0)
 			(effects
@@
 		)
 		(instances
-			(project ""
+			(project "R3M1XXX"
 				(path "/734751e6-bef2-4814-98c0-5802ec8506b2/1f2cf491-dbdb-4a6a-9515-9e3b3af8ab6f"
 					(reference "J1")
@@
 			)
 		)
-		(property "Value" "Conn_01x04"
+		(property "Value" "Conn_B2"
 			(at 125.73 161.2899 0)
 			(effects
@@
 		)
 		(instances
-			(project ""
+			(project "R3M1XXX"
 				(path "/734751e6-bef2-4814-98c0-5802ec8506b2/1f2cf491-dbdb-4a6a-9515-9e3b3af8ab6f"
 					(reference "J4")
@@
 		)
 		(instances
-			(project ""
+			(project "R3M1XXX"
 				(path "/734751e6-bef2-4814-98c0-5802ec8506b2/1f2cf491-dbdb-4a6a-9515-9e3b3af8ab6f"
 					(reference "U3")
@@
 			)
 		)
-		(property "Value" "Conn_01x06"
+		(property "Value" "Conn_B4"
 			(at 158.75 157.4799 0)
 			(effects
@@
 		)
 		(instances
-			(project ""
+			(project "R3M1XXX"
 				(path "/734751e6-bef2-4814-98c0-5802ec8506b2/1f2cf491-dbdb-4a6a-9515-9e3b3af8ab6f"
 					(reference "D1")
