File: KiCAD/X01/fx.kicad_sch (KiCad schematic)
At the start: 40 parts, among them SW10 SW, SW11 SW, SW12 SW, SW5 SW, SW6 SW, SW7 SW, SW8 SW, SW9 SW

Commit message: M01 & X01
Parts:
- added J5: Conn_A1, symbol Connector_Generic:Conn_01x06
- added J6: Conn_A2, symbol Connector_Generic:Conn_01x06
- added U4, U5: CD74HC4067M, Package_SO:SOIC-24W_7.5x15.4mm_P1.27mm, symbol 74xx:CD74HC4067M
Connections:
- net +5V: now also J5.2 (Pin_2), J6.2 (Pin_2), U4.24 (VCC), U5.24 (VCC)
- net FXSW1: now also U5.9 (I0)
- net FXSW2: now also U5.8 (I1)
- net FXSW3: now also U5.7 (I2)
- net FXSW4: now also U5.6 (I3)
- net FXSW5: now also U5.5 (I4)
- net FXSW6: now also U5.4 (I5)
- net FXSW7: now also U5.3 (I6)
- net FXSW8: now also U5.2 (I7)
- net GND: now also J5.1 (Pin_1), J6.1 (Pin_1), U4.12 (GND), U4.15 (~{E}), U5.12 (GND), U5.15 (~{E})
- net NP1IN: now also J6.5 (Pin_5)
- net NP1OUT: now also J6.6 (Pin_6)
- net POT1: now also U4.9 (I0)
- net POT2: now also U4.8 (I1)
- net POT3: now also U4.7 (I2)
- net POT5: now also U4.5 (I4)
- net POT6: now also U4.4 (I5)
- net POT7: now also U4.3 (I6)
- net POT4: now reaches RV4.2
- net POT4: now also U4.6 (I3)
- net POT8: now reaches RV8.2
- net POT8: now also U4.2 (I7)
- new net MPLEX-AP: J6.3 (Pin_3), U4.1 (COM)
- new net MPLEX-AS: J6.4 (Pin_4), U5.1 (COM)
- new net MPLEX-S0: J5.3 (Pin_3), U4.10 (S0), U5.10 (S0)
- new net MPLEX-S1: J5.4 (Pin_4), U4.11 (S1), U5.11 (S1)
- new net MPLEX-S2: J5.5 (Pin_5), U4.14 (S2), U5.14 (S2)
- new net MPLEX-S3: J5.6 (Pin_6), U4.13 (S3), U5.13 (S3)
- no-connect marks 0 -> 16
