File: KiCAD/M01/eq_pots.kicad_sch (KiCad schematic)
At the start: 14 parts, among them J4 Conn_01x04, J5 Conn_01x03, U5 CD74HC4067M

Commit message: M01 fixes
Parts:
- J3: renamed from J4; footprint (none) -> Connector_PinHeader_2.54mm:PinHeader_1x04_P2.54mm_Vertical
- J4: renamed from J5; footprint (none) -> Connector_PinHeader_2.54mm:PinHeader_1x03_P2.54mm_Vertical
- RV1, RV2, RV3, RV4: footprint (none) -> Potentiometer_THT:Potentiometer_Bourns_PTV09A-1_Single_Vertical
- RV10: renamed from RV7; footprint (none) -> Potentiometer_THT:Potentiometer_Bourns_PTV09A-1_Single_Vertical
- RV11: renamed from RV8; footprint (none) -> Potentiometer_THT:Potentiometer_Bourns_PTV09A-1_Single_Vertical
- RV5: renamed from RV9; footprint (none) -> Potentiometer_THT:Potentiometer_Bourns_PTV09A-1_Single_Vertical
- RV6: renamed from RV10; footprint (none) -> Potentiometer_THT:Potentiometer_Bourns_PTV09A-1_Single_Vertical
- RV7: renamed from RV11; footprint (none) -> Potentiometer_THT:Potentiometer_Bourns_PTV09A-1_Single_Vertical
- RV8: renamed from RV5; footprint (none) -> Potentiometer_THT:Potentiometer_Bourns_PTV09A-1_Single_Vertical
- RV9: renamed from RV6; footprint (none) -> Potentiometer_THT:Potentiometer_Bourns_PTV09A-1_Single_Vertical
Connections:
- net GND: now also RV7.3

Commit message: m01
Parts:
- added H10, H11, H5, H6, H7, H8, H9: MountingHole, MountingHole:MountingHole_3.2mm_M3, symbol Mechanical:MountingHole
Connections:
- net POT-C1: now also U5.18 (I13); no longer U5.5 (I4)
- net POT-L1: now also U5.17 (I14); no longer U5.9 (I0)
- net POT-L2: now also U5.16 (I15); no longer U5.8 (I1)
- net POT-R1: now also U5.19 (I12); no longer U5.2 (I7)
- net POT-R2: now also U5.21 (I10); no longer U5.23 (I8)
- net POT-R4: now also U5.5 (I4); no longer U5.21 (I10)
