File: KiCAD/M01/M01.kicad_pcb (KiCad board)
At the start: 2 copper layers, 236.4 x 106 mm, 159 parts, among them J1 Conn_01x05, J2 Conn_01x05, J3 Conn_01x04, J4 Conn_01x03, J5 Conn_B1, J6 Conn_B2, J7 Conn_01x03, J8 Conn_01x06, SW1 SW, SW2 SW, SW3 SW, SW4 SW, SW5 SW, U1 74HC595, U10 CD74HC4067M, U2 74HC595, U3 74HC595, U4 74HC595, U5 CD74HC4067M, U6 CD74HC4067M, U7 74HC595, U8 74HC595, U9 SR1-ML

Commit message: pots
Parts:
- RV14, RV15: footprint Potentiometer_THT:Potentiometer_Bourns_PTV09A-1_Single_Vertical -> PCM_Potentiometer_THT_US_AKL:Potentiometer_Bourns_PTA4543_Single_Slide
- moved RV14 191.5 mm to (-87.5, -31.2)

Commit message: m01
Parts:
- added D49: RCUED, LED_THT:LED_Rectangular_W3.9mm_H1.8mm, F.Cu at (234.0, 163.5)
- added R54: RCUER, Resistor_SMD:R_1206_3216Metric_Pad1.30x1.75mm_HandSolder, B.Cu at (233.5, 167.5)
- C4, C5, R31, R32, R33, R34, R35, R36, R52, R53, U10, U8, U9: moved to B.Cu
- D31, D32, D33: footprint LED_SMD:LED_1206_3216Metric_Pad1.42x1.75mm_HandSolder -> LED_THT:LED_Rectangular_W3.9mm_H1.8mm
- D34, D35, D36, D37, D38, D39, D40: value VUMLD -> VUCH1
- D41: value VUMLD -> LCUED; footprint LED_THT:LED_D3.0mm -> LED_THT:LED_Rectangular_W3.9mm_H1.8mm
- D42, D43, D44, D45, D46, D47, D48: value VUMLD -> VUCH2
- J7: footprint Connector_PinHeader_2.54mm:PinHeader_1x03_P2.54mm_Horizontal -> Connector_PinHeader_2.54mm:PinHeader_1x03_P2.54mm_Vertical
- R37, R38, R39, R40, R41, R42, R43: value VUMLR -> VUCH1L; moved to B.Cu
- R44: value VUMLR -> LCUER; moved to B.Cu
- R45, R46, R47, R48, R49, R50, R51: value VUMLR -> VUCH2R; moved to B.Cu
- RV14, RV15: footprint PCM_Potentiometer_THT_US_AKL:Potentiometer_Bourns_PTA4543_Single_Slide -> slider:SC6080GH
- moved RV15 451.8 mm to (241.5, 212.5)
- moved D34 434.7 mm to (197.8, 229.2), turned to 180 degrees
- moved D43 430.8 mm to (217.8, 223.6), turned to 180 degrees
- moved D42 428.6 mm to (217.8, 229.1), turned to 180 degrees
- moved D35 424.8 mm to (197.8, 223.6), turned to 180 degrees
- moved D44 420.9 mm to (217.8, 218.0), turned to 180 degrees
- moved D37 417.2 mm to (197.8, 212.5), turned to 180 degrees
- moved R45 415.6 mm to (222.0, 229.0), turned to 180 degrees
- moved R37 415.2 mm to (202.0, 229.0), turned to 180 degrees
- moved D36 415.0 mm to (197.8, 218.1), turned to 180 degrees
- moved D46 413.3 mm to (217.8, 206.9), turned to 180 degrees
- moved D45 411.2 mm to (217.8, 212.5), turned to 180 degrees
- moved R46 407.9 mm to (222.0, 223.5), turned to 180 degrees
- moved D38 407.3 mm to (197.8, 206.9), turned to 180 degrees
- moved R38 407.3 mm to (202.0, 223.5), turned to 180 degrees
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Connections:
- net LVU-LATCH renamed /Channels/LVU-LATCH
- net LVU-SIG renamed /Channels/LVU-SIG
- net MPLEX-D renamed /Channels/MPLEX-D
- net POT-LC renamed /Channels/POT-LC
- net POT-RC renamed /Channels/POT-RC
- net RVU-LATCH renamed /Channels/RVU-LATCH
- net RVU-SIG renamed /Channels/RVU-SIG
- net SW-LC renamed /Channels/SW-LC
- net SW-RC renamed /Channels/SW-RC
- J7 pad 3: SRCLK -> /Channels/SRCLK
- U10 pad 10: MPLEX-S0 -> /Channels/MPLEX-S0
- U10 pad 11: MPLEX-S1 -> /Channels/MPLEX-S1
- U10 pad 13: MPLEX-S3 -> /Channels/MPLEX-S3
- U10 pad 14: MPLEX-S2 -> /Channels/MPLEX-S2
- U8 pad 11: SRCLK -> /Channels/SRCLK
- U8 pad 7: unconnected-(U8-QH-Pad7) -> Net-(D49-A)
- U9 pad 11: SRCLK -> /Channels/SRCLK
Routing:
- net +5V: track 575.9 -> 717.7 mm
- net /Channels/SRCLK: track 0.00 -> 88.2 mm, vias 0 -> 3
- net Net-(D42-A): track 0.00 -> 70.8 mm
- net Net-(D41-A): track 0.00 -> 65.7 mm, vias 0 -> 2
- net /Channels/RVU-LATCH: track 0.00 -> 65.4 mm, vias 0 -> 2
- net /Channels/RVU-SIG: track 0.00 -> 64.2 mm, vias 0 -> 2
- net /Channels/SW-RC: track 0.00 -> 63.0 mm
- net /Channels/SW-LC: track 0.00 -> 57.0 mm
- net Net-(D34-A): track 0.00 -> 51.0 mm, vias 0 -> 2
- net Net-(D43-A): track 0.00 -> 47.7 mm
- net /Channels/LVU-SIG: track 0.00 -> 43.4 mm
- net /Channels/LVU-LATCH: track 0.00 -> 43.4 mm
- net Net-(D36-A): track 0.00 -> 43.2 mm
- net Net-(D44-A): track 0.00 -> 41.3 mm
- net Net-(D37-A): track 0.00 -> 38.0 mm
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Other:
- board size 236.4 x 106 mm -> 236.4 x 229 mm
