File: KiCAD/M01/channels.kicad_sch (KiCad schematic)
At the start: 43 parts, among them J7 Conn_01x03, J8 Conn_01x06, SW4 SW, SW5 SW, U10 CD74HC4067M, U8 SR1-ML, U9 74HC595

Commit message: M01 fixes
Parts:
- C4, C5: footprint (none) -> Capacitor_SMD:C_1206_3216Metric_Pad1.33x1.80mm_HandSolder
- D34, D35: footprint Library:LED_RED -> LED_THT:LED_D3.0mm
- D36, D37, D38, D39: footprint Library:LED_YELLOW -> LED_THT:LED_D3.0mm
- D40, D41, D42, D43, D44, D45, D46, D47, D48: footprint Library:LED_GREEN -> LED_THT:LED_D3.0mm
- J7: footprint (none) -> Connector_PinHeader_2.54mm:PinHeader_1x03_P2.54mm_Horizontal
- J8: footprint (none) -> Connector_PinHeader_2.54mm:PinHeader_1x06_P2.54mm_Vertical
- R52, R53: footprint (none) -> Resistor_SMD:R_1206_3216Metric_Pad1.30x1.75mm_HandSolder
- RV14, RV15: footprint (none) -> Potentiometer_THT:Potentiometer_Bourns_PTV09A-1_Single_Vertical
- SW4, SW5: footprint (none) -> Button_Switch_THT:SW_PUSH_6mm_H9.5mm
- U8: renamed from U9; footprint (none) -> Package_SO:SOIC-16W_5.3x10.2mm_P1.27mm
- renumbered R34 to R37, R35 to R38, R36 to R39, U8 to U9
Connections:
- no-connect marks 14 -> 15
Other:
- moved on the sheet: D34, D36, D38, D40, D43, D45, R37, R38, R39, R40, R41, R42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

Commit message: pots
Parts:
- RV14, RV15: footprint Potentiometer_THT:Potentiometer_Bourns_PTV09A-1_Single_Vertical -> PCM_Potentiometer_THT_US_AKL:Potentiometer_Bourns_PTA4543_Single_Slide
Changed lines of the file:
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@@
 			)
 		)
-		(property "Footprint" "Potentiometer_THT:Potentiometer_Bourns_PTV09A-1_Single_Vertical"
+		(property "Footprint" "PCM_Potentiometer_THT_US_AKL:Potentiometer_Bourns_PTA4543_Single_Slide"
 			(at 144.78 64.77 0)
 			(effects
@@
 		(on_board yes)
 		(dnp no)
-		(fields_autoplaced yes)
 		(property "Reference" "RV14"
 			(at 142.24 40.6399 0)
@@
 			)
 		)
-		(property "Footprint" "Potentiometer_THT:Potentiometer_Bourns_PTV09A-1_Single_Vertical"
-			(at 144.78 41.91 0)
-			(effects
-				(font
-					(size 1.27 1.27)
-				)
-				(hide yes)
-			)
-		)
+		(property "Footprint" "PCM_Potentiometer_THT_US_AKL:Potentiometer_Bourns_PTA4543_Single_Slide"
+			(at 144.78 27.686 0)
+			(effects
+				(font
+					(size 1.27 1.27)
+				)
+			)
+		)

Commit message: m01
Parts:
- added D49: RCUED, LED_THT:LED_Rectangular_W3.9mm_H1.8mm, symbol Device:LED_Filled
- added R54: RCUER, Resistor_SMD:R_1206_3216Metric_Pad1.30x1.75mm_HandSolder, symbol Device:R_Small
- D34, D35, D36, D37, D38, D39, D40: value VUMLD -> VUCH1
- D41: value VUMLD -> LCUED; footprint LED_THT:LED_D3.0mm -> LED_THT:LED_Rectangular_W3.9mm_H1.8mm
- D42, D43, D44, D45, D46, D47, D48: value VUMLD -> VUCH2
- J7: footprint Connector_PinHeader_2.54mm:PinHeader_1x03_P2.54mm_Horizontal -> Connector_PinHeader_2.54mm:PinHeader_1x03_P2.54mm_Vertical
- R37, R38, R39, R40, R41, R42, R43: value VUMLR -> VUCH1L
- R44: value VUMLR -> LCUER
- R45, R46, R47, R48, R49, R50, R51: value VUMLR -> VUCH2R
- RV14, RV15: footprint PCM_Potentiometer_THT_US_AKL:Potentiometer_Bourns_PTA4543_Single_Slide -> slider:SC6080GH
Connections:
- net GND: now also R54.1
- net at U8.7 (QH): now also D49.2 (A)
- new net: D49.1 (K), R54.2
- no-connect marks 15 -> 14
