File: KiCAD/M01/filters.kicad_sch (KiCad schematic)
At the start: 21 parts, among them J3 Conn_B1, J6 Conn_B2, SW1 SW, SW2 SW, SW3 SW, U6 74HC595, U7 CD74HC4067M

Commit message: M01 fixes
Parts:
- C1, C2, C3: footprint (none) -> Capacitor_SMD:C_1206_3216Metric_Pad1.33x1.80mm_HandSolder
- J5: renamed from J3; footprint (none) -> Connector_PinHeader_2.54mm:PinHeader_1x06_P2.54mm_Vertical
- J6: footprint (none) -> Connector_PinHeader_2.54mm:PinHeader_1x06_P2.54mm_Vertical
- R31, R32: footprint (none) -> Resistor_SMD:R_1206_3216Metric_Pad1.30x1.75mm_HandSolder
- R33: renamed from R37; footprint (none) -> Resistor_SMD:R_1206_3216Metric_Pad1.30x1.75mm_HandSolder
- R34: renamed from R38; footprint (none) -> Resistor_SMD:R_1206_3216Metric_Pad1.30x1.75mm_HandSolder
- R35: renamed from R39; footprint (none) -> Resistor_SMD:R_1206_3216Metric_Pad1.30x1.75mm_HandSolder
- R36: renamed from R33; footprint (none) -> Resistor_SMD:R_1206_3216Metric_Pad1.30x1.75mm_HandSolder
- RV12, RV13: footprint (none) -> Potentiometer_THT:Potentiometer_Bourns_PTV09A-1_Single_Vertical
- SW1, SW2, SW3: footprint (none) -> Button_Switch_THT:SW_PUSH_6mm_H9.5mm
- U7: renamed from U6; footprint (none) -> Package_SO:SOIC-16W_5.3x10.2mm_P1.27mm
- renumbered U7 to U6
Connections:
- net at R35.2: now also D33.2 (A)

Commit message: m01
Parts:
- added H12, H13, H14, H15: MountingHole, MountingHole:MountingHole_3.2mm_M3, symbol Mechanical:MountingHole

Commit message: m01
Parts:
- D31, D32, D33: footprint LED_SMD:LED_1206_3216Metric_Pad1.42x1.75mm_HandSolder -> LED_THT:LED_Rectangular_W3.9mm_H1.8mm
Changed lines of the file:
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@@
 			)
 		)
-		(property "Footprint" "LED_SMD:LED_1206_3216Metric_Pad1.42x1.75mm_HandSolder"
+		(property "Footprint" "LED_THT:LED_Rectangular_W3.9mm_H1.8mm"
 			(at 158.75 91.44 0)
 			(effects
@@
 			)
 		)
-		(property "Footprint" "LED_SMD:LED_1206_3216Metric_Pad1.42x1.75mm_HandSolder"
+		(property "Footprint" "LED_THT:LED_Rectangular_W3.9mm_H1.8mm"
 			(at 158.75 83.82 0)
 			(effects
@@
 			)
 		)
-		(property "Footprint" "LED_SMD:LED_1206_3216Metric_Pad1.42x1.75mm_HandSolder"
+		(property "Footprint" "LED_THT:LED_Rectangular_W3.9mm_H1.8mm"
 			(at 158.75 99.06 0)
 			(effects
