File: KiCAD/X01/FX-Pots/FX-Pots.kicad_pcb (KiCad board)
At the start: 2 copper layers, 50 x 108 mm, 28 parts, among them J1 Conn_01x05, J2 Conn_01x05, SW1 SW_Push_LED, SW2 SW_Push_LED, SW3 SW_Push_LED, SW4 SW_Push_LED, U1 74HC595, U2 CD74HC4067M

Commit message: pots rfx
Parts:
- moved J1 42.7 mm to (87.4, 125.0), turned to 90 degrees
- moved J2 35.2 mm to (86.4, 69.5), turned to 90 degrees
- moved H1 21.6 mm to (78.0, 65.1)
- moved H4 19.7 mm to (78.0, 124.0)
- moved RV4 14.9 mm to (103.5, 131.0), turned to -90 degrees
- moved U2 11.5 mm to (106.0, 96.5)
- moved R1 7.81 mm to (87.5, 50.5), turned to -90 degrees
- moved R5 6.80 mm to (86.5, 57.0)
- moved U1 3.35 mm to (81.5, 96.5)
- moved H2 2.31 mm to (108.0, 65.1)
- moved H3 2.02 mm to (108.0, 124.0)
Routing:
- net +5V: track 288.1 -> 0.00 mm
- net GND: track 254.1 -> 0.00 mm, vias 3 -> 0
- net FXSW4: track 71.3 -> 0.00 mm
- net FXSW1: track 63.7 -> 0.00 mm
- net FX-LED-4: track 60.3 -> 0.00 mm, vias 2 -> 0
- net FX-LED-1: track 55.0 -> 0.00 mm
- net POT4: track 54.3 -> 0.00 mm
- net POT1: track 43.9 -> 0.00 mm
- net FXSW2: track 33.2 -> 0.00 mm
- net FXSW3: track 33.2 -> 0.00 mm
- net FX-LED-3: track 31.7 -> 0.00 mm, vias 2 -> 0
- net MPLEX-AP: track 28.1 -> 0.00 mm
- net POT3: track 23.9 -> 0.00 mm
- net MPLEX-S0: track 15.3 -> 0.00 mm
- net MPLEX-S2: track 15.0 -> 0.00 mm
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Other:
- board size 50 x 108 mm -> 50 x 100 mm
