File: KiCAD/X01/FX-Pots/FX-Pots.kicad_sch (KiCad schematic)
At the start: 17 parts, among them J1 Conn_01x04, J2 Conn_01x03, U1 CD74HC4067M

Commit message: fx pots
Parts:
- removed H5, H6: MountingHole_M3, MountingHole:MountingHole_3.2mm_M3, symbol PCM_SL_Mechanical:MountingHole_M3
- removed J1: Conn_01x04, Connector_PinHeader_2.54mm:PinHeader_1x04_P2.54mm_Vertical, symbol Connector_Generic:Conn_01x04
- removed J2: Conn_01x03, Connector_PinHeader_2.54mm:PinHeader_1x03_P2.54mm_Vertical, symbol Connector_Generic:Conn_01x03
- removed RV5, RV6, RV7, RV8: R_Pot, Potentiometer_THT:Potentiometer_Bourns_PTV09A-1_Single_Vertical, symbol Device:R_Potentiometer_Small
- added C1, C2, C3, C4: 1uF, Capacitor_SMD:C_1206_3216Metric_Pad1.33x1.80mm_HandSolder, symbol Device:C_Small
- added J1, J2: Conn_01x05, Connector_PinSocket_2.54mm:PinSocket_1x05_P2.54mm_Vertical, symbol Connector_Generic:Conn_01x05
- added R1, R2, R3, R4: 220, PCM_Resistor_SMD_AKL:R_1206_3216Metric_Pad1.30x1.75mm_HandSolder, symbol Device:R_Small
- added R5, R6, R7, R8: 10K, PCM_Resistor_SMD_AKL:R_1206_3216Metric_Pad1.30x1.75mm_HandSolder, symbol Device:R_Small
- added SW1, SW2, SW3, SW4: SW_Push_LED, led-switch:SW_PUSH_6mm_LED, symbol Switch:SW_Push_LED
- added U1: 74HC595, Package_SO:SOIC-16_3.9x9.9mm_P1.27mm, symbol 74xx:74HC595
- renumbered U1 to U2
Connections:
- net +5V: now also J2.2 (Pin_2), R5.1, R6.1, R7.1, R8.1, U1.10 (~{SRCLR}), U1.16 (VCC)
- net GND: now also C1.2, C2.2, C3.2, C4.2, J2.1 (Pin_1), R1.1, R2.1, R3.1, R4.1, SW1.1, SW2.1, SW3.1, SW4.1, U1.13 (~{OE}), U1.8 (GND)
- net MPLEX-AP: now also J1.3 (Pin_3)
- net MPLEX-S0: now also J1.1 (Pin_1)
- net MPLEX-S1: now also J1.2 (Pin_2)
- net MPLEX-S2: now also J1.4 (Pin_4)
- net MPLEX-S3: now also J1.5 (Pin_5)
- net POT1: now also U2.7 (I2); no longer U2.18 (I13)
- net POT2: now also U2.8 (I1); no longer U2.17 (I14)
- net POT3: now also U2.17 (I14); no longer U2.8 (I1)
- net POT4: now also U2.18 (I13); no longer U2.7 (I2)
- net POT5 renamed FXSW4
- net FXSW4: now also C4.1, R8.2, SW4.2
- net POT6 renamed FXSW3
- net FXSW3: now also C3.1, R7.2, SW3.2
- net POT7 renamed FXSW2
- net FXSW2: now also C2.1, R6.2, SW2.2
- net POT8 renamed FXSW1
- net FXSW1: now also C1.1, R5.2, SW1.2
- new net: R3.2, SW3.3 (K)
- new net: R2.2, SW2.3 (K)
- new net: R1.2, SW1.3 (K)
- new net: R4.2, SW4.3 (K)
- new net FX-LED-1: SW1.4 (A), U1.2 (QC)
- new net FX-LED-2: SW2.4 (A), U1.3 (QD)
- new net FX-LED-3: SW3.4 (A), U1.4 (QE)
- new net FX-LED-4: SW4.4 (A), U1.5 (QF)
- new net FX-LED-LATCH: J2.4 (Pin_4), U1.12 (RCLK)
- new net FX-LED-SIG: J2.5 (Pin_5), U1.14 (SER)
- new net SRCLK: J2.3 (Pin_3), U1.11 (SRCLK)
- no-connect marks 8 -> 13
Other:
- moved on the sheet: U2

Commit message: pots rfx
Parts:
- SW1, SW2, SW3, SW4: footprint led-switch:SW_PUSH_6mm_LED -> led-sw:led switch
Changed lines of the file:
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@@
 	(wire
 		(pts
-			(xy 250.19 27.94) (xy 250.19 29.21)
-		)
-		(stroke
-			(width 0)
-			(type default)
-		)
-	)
-	(wire
-		(pts
 			(xy 209.55 88.9) (xy 213.36 88.9)
 		)
@@
 	(wire
 		(pts
+			(xy 250.19 119.38) (xy 250.19 120.65)
+		)
+		(stroke
+			(width 0)
+			(type default)
+		)
+	)
+	(wire
+		(pts
 			(xy 36.83 106.68) (xy 36.83 107.95)
 		)
@@
 	(wire
 		(pts
-			(xy 250.19 119.38) (xy 250.19 120.65)
+			(xy 250.19 27.94) (xy 250.19 29.21)
 		)
 		(stroke
@@
 			)
 		)
-		(property "Footprint" "led-switch:SW_PUSH_6mm_LED"
+		(property "Footprint" "led-sw:led switch"
 			(at 226.06 107.95 0)
 			(effects
@@
 		)
 		(instances
-			(project ""
+			(project "FX-Pots"
 				(path "/785e7457-0738-4da0-a9ef-90f983e5f9cc"
 					(reference "J1")
@@
 			)
 		)
-		(property "Footprint" "led-switch:SW_PUSH_6mm_LED"
+		(property "Footprint" "led-sw:led switch"
 			(at 226.06 55.88 0)
 			(effects
@@
 			)
 		)
-		(property "Footprint" "led-switch:SW_PUSH_6mm_LED"
+		(property "Footprint" "led-sw:led switch"
 			(at 226.06 81.28 0)
 			(effects
@@
 			)
 		)
-		(property "Footprint" "led-switch:SW_PUSH_6mm_LED"
+		(property "Footprint" "led-sw:led switch"
 			(at 226.06 30.48 0)
 			(effects
@@
 		)
 		(instances
-			(project ""
+			(project "FX-Pots"
 				(path "/785e7457-0738-4da0-a9ef-90f983e5f9cc"
 					(reference "SW1")
@@
 		)
 		(instances
-			(project ""
+			(project "FX-Pots"
 				(path "/785e7457-0738-4da0-a9ef-90f983e5f9cc"
 					(reference "U1")
