File: KiCAD/X01/Encoders-LCD/Encoders-LCD.kicad_pcb (KiCad board)
At the start: 2 copper layers, 110 x 76 mm, 35 parts, among them J1 Conn_B1, J2 Conn_B4, J3 Conn_B3, SW1 RotaryEncoder_Switch, SW2 RotaryEncoder_Switch, SW3 RotaryEncoder_Switch, SW4 SW_Push_LED, U1 ST7789, U2 CD74HC4067M, U3 ST7789

Commit message: deck btns
Parts:
- U1, U3: footprint Display-oled:RGB_096 -> Display-oled:1.14 7789
- moved U3 9.06 mm to (135.5, 68.6)
- moved U1 8.72 mm to (65.5, 68.5)
Routing:
- net GND: track 199.2 -> 236.4 mm
- net 3V3: track 151.4 -> 140.8 mm
- net SPI0_TX: track 10.1 -> 5.83 mm
- net SPI0_CS: track 10.1 -> 5.83 mm
- net SPI0_RX: track 10.1 -> 5.83 mm
- net SPI1_SCK: track 22.8 -> 18.8 mm
- net SPI1_RX: track 9.83 -> 5.90 mm
- net SPI1_TX: track 9.83 -> 5.91 mm
- net SPI1_CS: track 9.83 -> 5.91 mm
- net SPI0_SCK: track 22.7 -> 18.8 mm
