File: KiCAD/X01/Encoders-LCD/Encoders-LCD.kicad_sch (KiCad schematic)
At the start: 35 parts, among them J1 Conn_B1, J2 Conn_B4, J3 Conn_B3, SW1 RotaryEncoder_Switch, SW2 RotaryEncoder_Switch, SW3 RotaryEncoder_Switch, SW4 SW_Push_LED, U1 ST7789, U2 CD74HC4067M, U3 ST7789

Commit message: deck btns
Parts:
- U1, U3: footprint Display-oled:RGB_096 -> Display-oled:1.14 7789
Changed lines of the file:
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@@
 			)
 		)
-		(property "Footprint" "Display-oled:RGB_096"
+		(property "Footprint" "Display-oled:1.14 7789"
 			(at 121.666 130.81 0)
 			(effects
@@
 			)
 		)
-		(property "Footprint" "Display-oled:RGB_096"
+		(property "Footprint" "Display-oled:1.14 7789"
 			(at 164.846 130.81 0)
 			(effects
@@
 		)
 		(instances
-			(project ""
+			(project "Encoders-LCD"
 				(path "/094609a0-ed7a-433b-8808-fc69fd09a73b"
 					(reference "H1")
