File: KiCAD/0x01/Encoders-LCD/Encoders-LCD.kicad_sch (KiCad schematic)
At the start: 31 parts, among them J1 SIGNALS, J2 S_PINS, J3 DISPLAY_L, J4 DISPLAY_R, SW1 SW_Push_LED, SW2 RotaryEncoder_Switch, SW3 RotaryEncoder_Switch, SW4 RotaryEncoder_Switch, U1 74HC4051, U2 ST7789, U3 74HC4051, U4 ST7789

Commit message: encoders
Parts:
- removed J3: DISPLAY_L, Connector_Molex:Molex_KK-254_AE-6410-04A_1x04_P2.54mm_Vertical, symbol Connector_Generic:Conn_01x04
- removed J4: DISPLAY_R, Connector_Molex:Molex_KK-254_AE-6410-04A_1x04_P2.54mm_Vertical, symbol Connector_Generic:Conn_01x04
- removed U2, U4: ST7789, Display-oled:1.14 7789, symbol r3m1xxx_Library:ST7789-oled
- added J1: Conn_01x03, Connector_Molex:Molex_KK-254_AE-6410-03A_1x03_P2.54mm_Vertical, symbol Connector_Generic:Conn_01x03
- J2: renamed from J1; value SIGNALS -> MUX_A; footprint Connector_Molex:Molex_KK-254_AE-6410-04A_1x04_P2.54mm_Vertical -> Connector_Molex:Molex_KK-254_AE-6410-06A_1x06_P2.54mm_Vertical; symbol Connector_Generic:Conn_01x04 -> Connector_Generic:Conn_01x06
- J3: renamed from J2; value S_PINS -> MUX_B; footprint Connector_Molex:Molex_KK-254_AE-6410-04A_1x04_P2.54mm_Vertical -> Connector_Molex:Molex_KK-254_AE-6410-06A_1x06_P2.54mm_Vertical; symbol Connector_Generic:Conn_01x04 -> Connector_Generic:Conn_01x06
- renumbered U3 to U2
Connections:
- net GND: now also J3.1 (Pin_1), J1.1 (Pin_1)
- net SF-LED: now also J1.3 (Pin_3); no longer J3.4 (Pin_4)
- net SIG_B: now also J3.3 (Pin_3); no longer J2.4 (Pin_4)
- net VCC: now also J3.2 (Pin_2), J1.2 (Pin_2)
- removed net S0: J3.1 (Pin_1), U1.11 (S0), U2.11 (S0)
- removed net S1: J3.2 (Pin_2), U1.10 (S1), U2.10 (S1)
- removed net S2: J3.3 (Pin_3), U1.9 (S2), U2.9 (S2)
- new net S0A: J2.4 (Pin_4), U1.11 (S0)
- new net S0B: J3.4 (Pin_4), U2.11 (S0)
- new net S1A: J2.5 (Pin_5), U1.10 (S1)
- new net S1B: J3.5 (Pin_5), U2.10 (S1)
- new net S2A: J2.6 (Pin_6), U1.9 (S2)
- new net S2B: J3.6 (Pin_6), U2.9 (S2)
