File: KiCAD/0x01/Encoders-LCD/Encoders-LCD.kicad_pcb (KiCad board)
At the start: 2 copper layers, 100 x 76 mm, 29 parts, among them J1 I2C_Conn, J2 Conn_01x05, SW1 SW_SHIFT, SW2 SW_LEFT, SW3 SW_RIGHT, U4 A_REG, U5 B_REG, U6 SW_REG

Commit message: wiring encoders
Parts:
- moved J1 8.11 mm to (86.1, 85.3), turned to 90 degrees
- moved C2 8.03 mm to (93.7, 81.3)
Routing:
- net GND: track 294.5 -> 364.2 mm, vias 25 -> 26
- net /B3: track 29.6 -> 94.6 mm
- net /A3: track 119.9 -> 65.6 mm, vias 4 -> 2
- net /SER_A: track 135.5 -> 100.8 mm
- net /RSW: track 96.5 -> 74.1 mm
- net /B2: track 89.0 -> 73.6 mm
- net VCC: track 376.5 -> 363.4 mm, vias 6 -> 18
- net /A1: track 38.4 -> 29.7 mm, vias 0 -> 2
- net /SW1: track 175.0 -> 168.4 mm
- net /SFTSW: track 26.1 -> 32.6 mm
- net /PL: track 42.7 -> 46.4 mm, vias 2 -> 0
- net /SW3: track 59.5 -> 57.6 mm
- net /SER_S: track 21.9 -> 20.1 mm
- net /CLK: track 43.2 -> 45.0 mm, vias 0 -> 2
- net /LSW: track 123.1 -> 121.5 mm
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