File: KiCAD/0x01/Encoders-LCD/Encoders-LCD.kicad_pcb (KiCad board)
At the start: 2 copper layers, 100 x 76 mm, 32 parts, among them J1 Conn_01x04, J2 Conn_01x04, SW1 SW_LEFT, SW2 SW_SHIFT, SW3 SW_RIGHT, U1 ATtiny412-SS, U2 3631AS, U3 3631AS, U4 ATtiny412-SS, U5 HT16K33 24SOP, U6 ATtiny412-SS

Commit message: fixes
Parts:
- U5: footprint Package_SO:SSOP-24_5.3x8.2mm_P0.65mm -> Package_SO:SOP-24_7.5x15.4mm_P1.27mm
- moved C1 2.50 mm to (82.2, 79.1)
- moved D1 2.32 mm to (101.1, 84.5)
- moved U5 2.05 mm to (90.3, 89.4)
Routing:
- net VCC: track 111.3 -> 9.48 mm, vias 8 -> 2
- net GND: track 118.4 -> 17.0 mm, vias 5 -> 8
- net /SEG2: track 192.4 -> 104.2 mm, vias 2 -> 1
- net /SCL: track 212.5 -> 159.6 mm, vias 4 -> 2
- net /COM3: track 65.2 -> 38.3 mm
- net /SDA: track 172.9 -> 149.4 mm, vias 3 -> 0
- net /SEG1: track 113.2 -> 96.0 mm, vias 0 -> 1
- net /SEG3: track 111.5 -> 99.6 mm, vias 4 -> 1
- net /SEG5: track 76.3 -> 65.7 mm, vias 4 -> 3
- net Net-(D1-K): track 136.7 -> 128.8 mm, vias 7 -> 1
- net /SEG4: track 73.7 -> 67.6 mm, vias 4 -> 1
- net /COM6: track 40.4 -> 35.9 mm, vias 0 -> 1
- net /SEG6: track 90.7 -> 86.4 mm, vias 3 -> 2
- net /COM1: track 50.0 -> 53.5 mm
- net /COM5: track 37.1 -> 34.6 mm, vias 0 -> 3
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
Commit message: lcd encoders
Parts:
- removed the C3 at (55.3, 100.8)
- removed J2: Conn_01x04, Connector_JST:JST_PH_S4B-PH-K_1x04_P2.00mm_Horizontal
- added C2: 10uF, Capacitor_SMD:C_0805_2012Metric_Pad1.18x1.45mm_HandSolder, B.Cu at (112.0, 100.5)
- added C7: 100nF, Capacitor_SMD:C_0603_1608Metric_Pad1.08x0.95mm_HandSolder, B.Cu at (55.5, 100.5)
- added C8: 100nF, Capacitor_SMD:C_0603_1608Metric_Pad1.08x0.95mm_HandSolder, F.Cu at (85.6, 78.7)
- C3: renamed from C2; value 10uF -> 100nF; footprint Capacitor_SMD:C_0805_2012Metric_Pad1.18x1.45mm_HandSolder -> Capacitor_SMD:C_0603_1608Metric_Pad1.08x0.95mm_HandSolder
- C4: value 10uF -> 100nF; footprint Capacitor_SMD:C_0805_2012Metric_Pad1.18x1.45mm_HandSolder -> Capacitor_SMD:C_0603_1608Metric_Pad1.08x0.95mm_HandSolder
- C5: moved to B.Cu
- moved C5 63.6 mm to (53.0, 100.5), turned to 90 degrees
- moved C6 29.5 mm to (83.1, 78.7), turned to 90 degrees
- moved C1 20.1 mm to (96.0, 64.5), turned to 0 degrees
- moved C4 1.11 mm to (114.5, 100.5), turned to 90 degrees
- moved C3 0.91 mm to (96.0, 62.3)
Routing:
- net VCC: track 9.48 -> 237.4 mm, vias 2 -> 7
- net Net-(D1-K): track 128.8 -> 202.5 mm, vias 1 -> 4
- net GND: track 17.0 -> 58.3 mm, vias 8 -> 4
- net /SDA: track 149.4 -> 178.2 mm, vias 0 -> 6
- net /SCL: track 159.6 -> 176.8 mm
- net /SEG6: track 86.4 -> 97.9 mm, vias 2 -> 5
- net /SEG3: track 99.6 -> 107.8 mm, vias 1 -> 2
- net /COM6: track 35.9 -> 41.0 mm, vias 1 -> 0
- net /SEG1: track 96.0 -> 100.9 mm, vias 1 -> 2
- net /COM5: track 34.6 -> 37.9 mm, vias 3 -> 0
- net /SEG2: track 104.2 -> 107.3 mm, vias 1 -> 5
- net /SEG7: track 74.8 -> 72.0 mm
- net /COM2: track 39.3 -> 41.9 mm
- net /COM4: track 27.8 -> 30.2 mm, vias 1 -> 0
- net /SEG5: track 65.7 -> 67.8 mm, vias 3 -> 2
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- added copper zone on B.Cu, net GND
- removed copper zone on B.Cu, net VCC
Other:
- board text added: "R3M1XXX 0x01 LCD-ENCODERS v1.3"

Commit message: pots fixed
Connections:
- SW1 pad 2: /SEG1 -> /SEG5
- SW2 pad 2: /SEG2 -> /SEG4
Routing:
- net /SEG4: track 65.7 -> 117.2 mm
- net /SEG5: track 67.8 -> 101.8 mm
- net /SEG2: track 107.3 -> 79.7 mm, vias 5 -> 3
- net /SEG1: track 100.9 -> 77.2 mm
Changed lines of the file:
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@@
 			(layers "*.Cu" "*.Mask")
 			(remove_unused_layers no)
-			(net 3 "/SEG1")
+			(net 25 "/SEG5")
 			(pinfunction "2")
 			(pintype "passive")
@@
 			(layers "*.Cu" "*.Mask")
 			(remove_unused_layers no)
-			(net 3 "/SEG1")
+			(net 25 "/SEG5")
 			(pinfunction "2")
 			(pintype "passive")
@@
 			(layers "*.Cu" "*.Mask")
 			(remove_unused_layers no)
-			(net 14 "/SEG2")
+			(net 27 "/SEG4")
 			(pinfunction "2")
 			(pintype "passive")
@@
 			(layers "*.Cu" "*.Mask")
 			(remove_unused_layers no)
-			(net 14 "/SEG2")
+			(net 27 "/SEG4")
 			(pinfunction "2")
 			(pintype "passive")
@@
 			(keep_text_aligned yes)
 		)
-		(gr_text "2992,1260 mils"
+		(gr_text "2992.1260 mils"
 			(at 152.52 82 90)
 			(layer "Eco2.User")
@@
 			(keep_text_aligned yes)
 		)
-		(gr_text "3937,0079 mils"
+		(gr_text "3937.0079 mils"
 			(at 89.999999 29.920278 1.145915576e-06)
 			(layer "Eco2.User")
@@
 	)
 	(segment
-		(start 54.991 68.072)
-		(end 54.14 67.221)
-		(width 0.2032)
-		(layer "F.Cu")
-		(net 3)
-	)
-	(segment
-		(start 57.3516 76.2216)
-		(end 57.3516 69.5436)
-		(width 0.2032)
-		(layer "F.Cu")
-		(net 3)
-	)
-	(segment
 		(start 91.186 78.994)
 		(end 97.5948 78.994)
@@
 		(net 3)
 	)
-	(segment
-		(start 55.88 68.072)
-		(end 54.991 68.072)
-		(width 0.2032)
-		(layer "F.Cu")
-		(net 3)
-	)
-	(segment
-		(start 54.14 67.221)
-		(end 54.14 60.85)
-		(width 0.2032)
-		(layer "F.Cu")
-		(net 3)
-	)
-	(segment
-		(start 57.3516 69.5436)
-		(end 55.88 68.072)
-		(width 0.2032)
-		(layer "F.Cu")
-		(net 3)
-	)
-	(segment
-		(start 54.14 60.85)
-		(end 60.64 60.85)
-		(width 0.2032)
-		(layer "F.Cu")
-		(net 3)
-	)
 	(via
 		(at 91.186 78.994)
@@
 	)
 	(segment
-		(start 81.407 96.52)
-		(end 81.407 87.503)
+		(start 67.5116 76.2216)
+		(end 67.5116 81.3324)
 		(width 0.2032)
 		(layer "F.Cu")
@@
 	)
 	(segment
-		(start 67.564 80.518)
-		(end 67.5116 80.4656)
+		(start 67.5116 81.3324)
+		(end 67.437 81.407)
 		(width 0.2032)
 		(layer "F.Cu")
@@
 		(net 14)
 	)
-	(segment
-		(start 67.5116 80.4656)
-		(end 67.5116 76.2216)
-		(width 0.2032)
-		(layer "F.Cu")
-		(net 14)
-	)
-	(via
-		(at 81.407 96.52)
-		(size 0.9)
-		(drill 0.4)
-		(layers "F.Cu" "B.Cu")
-		(net 14)
-	)
 	(via
 		(at 95.631 77.343)
@@
 	)
 	(via
-		(at 81.407 87.503)
+		(at 67.437 81.407)
 		(size 0.9)
 		(drill 0.4)
@@
 		(net 14)
 	)
-	(via
-		(at 67.564 80.518)
-		(size 0.9)
-		(drill 0.4)
-		(layers "F.Cu" "B.Cu")
-		(net 14)
-	)
-	(segment
-		(start 74.295 82.042)
-		(end 72.898 80.645)
-		(width 0.2032)
-		(layer "B.Cu")
-		(net 14)
-	)
-	(segment
-		(start 86.92 106.898)
-		(end 93.42 106.898)
-		(width 0.2032)
-		(layer "B.Cu")
-		(net 14)
-	)
-	(segment
-		(start 81.407 101.385)
-		(end 81.407 96.52)
-		(width 0.2032)
-		(layer "B.Cu")
-		(net 14)
-	)
 	(segment
 		(start 88.392 86.995)
@@
 	)
 	(segment
-		(start 72.898 80.645)
-		(end 67.691 80.645)
-		(width 0.2032)
-		(layer "B.Cu")
-		(net 14)
-	)
-	(segment
-		(start 74.295 83.82)
-		(end 74.295 82.042)
-		(width 0.2032)
-		(layer "B.Cu")
-		(net 14)
-	)
-	(segment
-		(start 76.581 87.503)
-		(end 74.803 85.725)
+		(start 76.2 87.503)
+		(end 85.647 87.503)
 		(width 0.2032)
 		(layer "B.Cu")
@@
 	)
 	(segment
-		(start 81.407 87.503)
-		(end 76.581 87.503)
+		(start 101.219 74.168)
+		(end 98.044 77.343)
 		(width 0.2032)
 		(layer "B.Cu")
@@
 	)
 	(segment
-		(start 101.219 74.168)
-		(end 98.044 77.343)
+		(start 91.313 80.772)
+		(end 90.297 80.772)
 		(width 0.2032)
 		(layer "B.Cu")
@@
 	)
 	(segment
-		(start 91.313 80.772)
-		(end 90.297 80.772)
+		(start 67.437 81.407)
+		(end 73.279 81.407)
 		(width 0.2032)
 		(layer "B.Cu")
@@
 	)
 	(segment
-		(start 86.92 106.898)
-		(end 81.407 101.385)
+		(start 73.914 82.042)
+		(end 73.914 85.217)
 		(width 0.2032)
 		(layer "B.Cu")
@@
 	)
 	(segment
-		(start 92.22 77.36)
-		(end 92.22 79.865)
+		(start 73.914 85.217)
+		(end 76.2 87.503)
 		(width 0.2032)
 		(layer "B.Cu")
@@
 	)
 	(segment
-		(start 67.691 80.645)
-		(end 67.564 80.518)
+		(start 92.22 77.36)
+		(end 92.22 79.865)
 		(width 0.2032)
 		(layer "B.Cu")
@@
 	)
 	(segment
-		(start 74.295 85.217)
-		(end 74.295 83.82)
-		(width 0.2032)
-		(layer "B.Cu")
-		(net 14)
-	)
-	(segment
 		(start 92.22 79.865)
 		(end 91.313 80.772)
@@
 	)
 	(segment
-		(start 85.647 87.503)
-		(end 81.407 87.503)
-		(width 0.2032)
-		(layer "B.Cu")
-		(net 14)
-	)
-	(segment
 		(start 90.297 80.772)
 		(end 88.392 82.677)
@@
 	)
 	(segment
-		(start 74.803 85.725)
-		(end 74.295 85.217)
+		(start 73.279 81.407)
+		(end 73.914 82.042)
 		(width 0.2032)
 		(layer "B.Cu")
@@
 	)
 	(segment
+		(start 52.07 83.64)
+		(end 52.07 62.92)
+		(width 0.2032)
+		(layer "F.Cu")
+		(net 25)
+	)
+	(segment
+		(start 54.8116 86.3816)
+		(end 52.07 83.64)
+		(width 0.2032)
+		(layer "F.Cu")
+		(net 25)
+	)
+	(segment
+		(start 54.14 60.85)
+		(end 60.64 60.85)
+		(width 0.2032)
+		(layer "F.Cu")
+		(net 25)
+	)
+	(segment
 		(start 92.837 90.932)
 		(end 113.284 90.932)
@@
 		(net 25)
 	)
+	(segment
+		(start 54.14 60.85)
+		(end 52.07 62.92)
+		(width 0.2032)
+		(layer "F.Cu")
+		(net 25)
+	)
 	(via
 		(at 113.284 90.932)
@@
 	)
 	(segment
+		(start 86.92 106.898)
+		(end 93.42 106.898)
+		(width 0.2032)
+		(layer "B.Cu")
+		(net 27)
+	)
+	(segment
+		(start 116.078 89.789)
+		(end 111.3248 94.5422)
+		(width 0.2032)
+		(layer "B.Cu")
+		(net 27)
+	)
+	(segment
+		(start 84.927 106.898)
+		(end 84.074 106.045)
+		(width 0.2032)
+		(layer "B.Cu")
+		(net 27)
+	)
+	(segment
+		(start 100.2758 94.5422)
+		(end 95.123 99.695)
+		(width 0.2032)
+		(layer "B.Cu")
+		(net 27)
+	)
+	(segment
+		(start 84.074 100.711)
+		(end 84.074 106.045)
+		(width 0.2032)
+		(layer "B.Cu")
+		(net 27)
+	)
+	(segment
 		(start 91.694 90.043)
 		(end 91.821 89.916)
@@
 	)
 	(segment
+		(start 86.92 106.898)
+		(end 84.927 106.898)
+		(width 0.2032)
+		(layer "B.Cu")
+		(net 27)
+	)
+	(segment
+		(start 95.123 99.695)
+		(end 85.09 99.695)
+		(width 0.2032)
+		(layer "B.Cu")
+		(net 27)
+	)
+	(segment
 		(start 85.647 90.043)
 		(end 91.694 90.043)
@@
 	)
 	(segment
+		(start 85.09 99.695)
+		(end 84.074 100.711)
+		(width 0.2032)
+		(layer "B.Cu")
+		(net 27)
+	)
+	(segment
 		(start 116.078 89.789)
 		(end 116.178 89.689)
@@
 		(width 0.2032)
 		(layer "B.Cu")
+		(net 27)
+	)
+	(segment
+		(start 111.3248 94.5422)
+		(end 100.2758 94.5422)
+		(width 0.2032)
+		(layer "B.Cu")
