File: KiCAD/0x01/FX-Pads/FX-Pads.kicad_pcb (KiCad board)
At the start: 2 copper layers, 100 x 100 mm, 36 parts, among them J1 CONTROL, J2 DATA, SW1 SW_Push, SW10 SW_Push, SW11 SW_Push, SW12 SW_Push, SW13 SW_Push, SW14 SW_Push, SW15 SW_Push, SW16 SW_Push, SW2 SW_Push, SW3 SW_Push, SW4 SW_Push, SW5 SW_Push, SW6 SW_Push, SW7 SW_Push, SW8 SW_Push, SW9 SW_Push, U1 CD74HC4067M

Commit message: pads
Parts:
- added H1: MountingHole, MountingHole:MountingHole_2mm, F.Cu at (125.0, 62.5)
- added H10: MountingHole, MountingHole:MountingHole_2mm, F.Cu at (62.5, 125.0)
- added H11: MountingHole, MountingHole:MountingHole_2mm, F.Cu at (87.5, 125.0)
- added H12: MountingHole, MountingHole:MountingHole_2mm, F.Cu at (125.0, 137.5)
- added H13: MountingHole, MountingHole:MountingHole_2mm, F.Cu at (75.0, 137.5)
- added H14: MountingHole, MountingHole:MountingHole_2mm, F.Cu at (125.0, 112.5)
- added H15: MountingHole, MountingHole:MountingHole_2mm, F.Cu at (112.5, 125.0)
- added H16: MountingHole, MountingHole:MountingHole_2mm, F.Cu at (137.5, 125.0)
- added H2: MountingHole, MountingHole:MountingHole_2mm, F.Cu at (137.5, 75.0)
- added H3: MountingHole, MountingHole:MountingHole_2mm, F.Cu at (125.0, 87.5)
- added H4: MountingHole, MountingHole:MountingHole_2mm, F.Cu at (75.0, 62.5)
- added H5: MountingHole, MountingHole:MountingHole_2mm, F.Cu at (87.5, 75.0)
- added H6: MountingHole, MountingHole:MountingHole_2mm, F.Cu at (112.5, 75.0)
- added H7: MountingHole, MountingHole:MountingHole_2mm, F.Cu at (75.0, 87.5)
- added H8: MountingHole, MountingHole:MountingHole_2mm, F.Cu at (62.5, 75.0)
- added H9: MountingHole, MountingHole:MountingHole_2mm, F.Cu at (75.0, 112.5)
Routing:
- net GND: track 39.6 -> 227.4 mm, vias 8 -> 34
- net VCC: track 331.1 -> 457.4 mm, vias 28 -> 33
- net Net-(U1-I11): track 177.2 -> 178.3 mm
- net /OUT: track 126.9 -> 127.5 mm

Commit message: fx pads gerbers
Parts:
- added H17: MountingHole, MountingHole:MountingHole_2.2mm_M2, F.Cu at (53.0, 53.0)
- added H18: MountingHole, MountingHole:MountingHole_2.2mm_M2, F.Cu at (147.0, 53.0)
- added H19: MountingHole, MountingHole:MountingHole_2.2mm_M2, F.Cu at (53.0, 147.0)
- added H20: MountingHole, MountingHole:MountingHole_2.2mm_M2, F.Cu at (147.0, 147.0)
- H1, H10, H11, H12, H13, H14, H15, H16, H2, H3, H4, H5, H6, H7, H8, H9: footprint MountingHole:MountingHole_2mm -> MountingHole:MountingHole_3.2mm_M3_ISO7380
- J1, J2: moved to B.Cu
- R1: footprint PCM_Resistor_SMD_AKL:R_0805_2012Metric_Pad1.20x1.40mm_HandSolder -> Resistor_SMD:R_0805_2012Metric_Pad1.20x1.40mm_HandSolder
- turned J1 to 90 degrees
- turned J2 to -90 degrees
Routing:
- net GND: track 227.4 -> 240.2 mm, vias 34 -> 36
- net Net-(U1-I14): track 138.3 -> 137.7 mm
- net Net-(U1-I15): track 116.3 -> 115.8 mm
- net VCC: vias 33 -> 27
Other:
- outline, holes or cut-outs redrawn
- board text added: "GND"
- board text added: "NP"
- board text added: "OUT"
- board text added: "S0"
- board text added: "S1"
- board text added: "S2"
- board text added: "S3"
- board text added: "VCC"
