File: DemoBox/lcd-ht16k33/lcd-ht16k33.kicad_sch (KiCad schematic)
At the start: 7 parts, among them U1 HT16K33 24SOP, U2 3631AS, U3 3631AS

Commit message: demo lcd ht16k33
Parts:
- added J1: Conn_01x04, Connector_Molex:Molex_KK-254_AE-6410-04A_1x04_P2.54mm_Vertical, symbol Connector_Generic:Conn_01x04
- C1: footprint Capacitor_SMD:C_0805_2012Metric_Pad1.18x1.45mm_HandSolder -> Capacitor_SMD:C_1206_3216Metric_Pad1.33x1.80mm_HandSolder
- U2, U3: footprint (none) -> sharedLibrary:3631AS
Connections:
- net GND: now also J1.1 (Pin_1)
- net SCL: now also J1.4 (Pin_4)
- net SDA: now also J1.3 (Pin_3)
- net VCC: now also J1.2 (Pin_2)

Commit message: refactor demobox
Parts:
- U1: footprint Package_SO:SSOP-24_5.3x8.2mm_P0.65mm -> Package_SO:SOP-24_7.5x15.4mm_P1.27mm
Changed lines of the file:
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@@
 			)
 		)
-		(property "Footprint" "Package_SO:SSOP-24_5.3x8.2mm_P0.65mm"
+		(property "Footprint" "Package_SO:SOP-24_7.5x15.4mm_P1.27mm"
 			(at 67.31 27.432 0)
 			(effects
