File: KiCAD/0x01/FX-Pots/FX-Pots.kicad_sch (KiCad schematic)
At the start: 41 parts, among them J1 IN, J2 OUT, SW1 SW_Push_LED, SW2 SW_Push_LED, SW3 SW_Push_LED, SW4 SW_Push_LED, SW5 SW_Push_LED, SW6 SW_Push_LED, SW7 SW_Push_LED, SW8 SW_Push_LED, U1 ADS7830, U2 HT16K33 24SOP

Commit message: fx-pots refactoring WIP
Parts:
- removed D3: 1N4148, Diode_SMD:D_SOD-323_HandSoldering, symbol Device:D_Small
- added R1: 5R, Resistor_SMD:R_0805_2012Metric_Pad1.20x1.40mm_HandSolder, symbol Device:R_Small
- C2: value 10uF -> 1uF; footprint Capacitor_SMD:C_0805_2012Metric_Pad1.18x1.45mm_HandSolder -> Capacitor_SMD:C_0603_1608Metric_Pad1.08x0.95mm_HandSolder
- C4: value 10uF -> 1uF
- D1, D2: footprint Diode_SMD:D_SOD-323_HandSoldering -> Diode_SMD:D_SOD-123F
- renumbered R1 to R2, R2 to R3, R5 to R4, R6 to R5, R3 to R6, R4 to R7
Connections:
- net +5V: now also R1.1; no longer C1.1, C2.1, U1.16 (VDD)
- net A0_H: no longer SW2.4 (A)
- net A1_H: no longer SW1.4 (A)
- net COM0: now also SW5.3 (K), SW6.3 (K), SW7.3 (K), SW8.3 (K)
- net COM1: no longer SW5.3 (K), SW6.3 (K), SW7.3 (K), SW8.3 (K)
- net R2: now also SW1.1, SW1.4 (A); no longer SW5.4 (A)
- net R3: now also SW2.1, SW2.4 (A); no longer SW1.1, SW6.4 (A)
- net R4: now also SW3.1; no longer SW2.1
- net R5: now also SW4.1; no longer SW3.1
- net R6: now also SW5.1, SW5.4 (A); no longer SW4.1, SW7.4 (A)
- net R7: now also SW6.1, SW6.4 (A); no longer SW5.1, SW8.4 (A)
- net R8: now also SW7.1, SW7.4 (A); no longer SW6.1
- net R9: now also SW8.1, SW8.4 (A); no longer SW7.1
- net at SW5.2, SW6.2, SW7.2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: now also D2.1 (K), SW1.2, SW2.2, SW3.2, SW4.2
- net COM2: no longer names the net of U2.4 (COM2/KS1)
- net R10: no longer names the net of U2.11 (ROW10/K9)
- net R10: no longer SW8.1
- new net: C1.1, C2.1, R1.2, U1.16 (VDD)
- no-connect marks 8 -> 10
Other:
- moved on the sheet: C1, C2, U1

Commit message: fxpots wip
Parts:
- removed J2: OUT, Connector_JST:JST_PH_S4B-PH-K_1x04_P2.00mm_Horizontal, symbol Connector_Generic:Conn_01x04
- added C5: 100nF, Capacitor_SMD:C_0603_1608Metric_Pad1.08x0.95mm_HandSolder, symbol Device:C_Small
- C4: footprint Capacitor_SMD:C_0805_2012Metric_Pad1.18x1.45mm_HandSolder -> Capacitor_SMD:C_0603_1608Metric_Pad1.08x0.95mm_HandSolder
- renumbered R2 to R1, R3 to R2, R1 to R3
Connections:
- net GND: now also C5.2
- net at C1.1, C2.1, R3.2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: now also U1.10 (REFin/REFout), C5.1
- no-connect marks 10 -> 9
Other:
- moved on the sheet: C3, C4, D1, J1, JP1, JP2, JP3, JP4, R1, R2, R4, R5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
