File: KiCAD/0x01/Controller-2040/Controller-2040.kicad_sch (KiCad schematic)
At the start: 3 parts, among them J1 pots-conn, J2 enc-conn

Commit message: rp2040 zero
Parts:
- added H1, H2, H3: MountingHole, MountingHole:MountingHole_3.2mm_M3, symbol Mechanical:MountingHole
- U1: renamed from A1; value RaspberryPi_Pico -> RP2040-ZERO; footprint Module:RaspberryPi_Pico_SMD -> 2040Library:MODULE_RP2040-ZEROa; symbol MCU_Module:RaspberryPi_Pico_Extensive -> 2040zero:RP2040-ZERO; Availability (none) -> Not in stock; Check_prices (none) -> https://www.snapeda.com/parts/RP2040-ZERO/Waveshare+Electro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; Description_1 (none) -> Low-Cost, High-Performance Pico-Like MCU Board Based On Ras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; MANUFACTURER (none) -> Waveshare; MAXIMUM_PACKAGE_HEIGHT (none) -> 5.35mm; MF (none) -> Waveshare Electronics; MP (none) -> RP2040-ZERO; PARTREV (none) -> NA; Package (none) -> Package; Price (none) -> None; STANDARD (none) -> Manufacturer Recommendations; SnapEDA_Link (none) -> https://www.snapeda.com/parts/RP2040-ZERO/Waveshare+Electro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
Connections:
- net GND: now also U1.22 (GND); no longer U1.13 (GND), U1.18 (GND), U1.23 (GND), U1.28 (GND), U1.3 (GND), U1.38 (GND), U1.8 (GND), U1.D2 (GND)
- net SCL: now also U1.6 (GP5); no longer U1.7 (GPIO5)
- net SDA: now also U1.5 (GP4); no longer U1.6 (GPIO4)
- net VCC: now also U1.23 (5V); no longer U1.40 (VBUS)
- no-connect marks 37 -> 19
