File: KiCAD/0x1F/EquBoard/EquBoard.kicad_pcb (KiCad board)
At the start: 2 copper layers, 150 x 100 mm, 30 parts, among them J1 MPLEX-IN, J2 MPLEX-OUT, J3 MPLEX-AP, J4 LED-CONN, SW1 SW_LED_1, SW2 SW_LED_2, U1 CD74HC4067M

Commit message: rp2040 zero
Parts:
- removed J2: MPLEX-OUT, Connector_PinHeader_2.54mm:PinHeader_1x04_P2.54mm_Vertical
- removed J3: MPLEX-AP, Connector_PinHeader_2.54mm:PinHeader_1x03_P2.54mm_Vertical
- removed J4: LED-CONN, Connector_PinHeader_2.54mm:PinHeader_1x02_P2.54mm_Vertical
- removed SW1: SW_LED_1, eqLibrary:led switch
- removed SW2: SW_LED_2, eqLibrary:led switch
- added C3: 10uF, Capacitor_SMD:C_0603_1608Metric_Pad1.08x0.95mm_HandSolder, F.Cu at (209.8, 79.2)
- added C4: 10uF, Capacitor_SMD:C_0805_2012Metric_Pad1.18x1.45mm_HandSolder, F.Cu at (210.0, 84.4)
- added C5: 1uF, Capacitor_SMD:C_0603_1608Metric_Pad1.08x0.95mm_HandSolder, F.Cu at (209.8, 81.7)
- added R3: 5R, Resistor_SMD:R_0805_2012Metric_Pad1.20x1.40mm_HandSolder, F.Cu at (209.9, 64.1)
- added R4: 10K, Resistor_SMD:R_0805_2012Metric_Pad1.20x1.40mm_HandSolder, F.Cu at (209.9, 67.0)
- added R5: 5R, Resistor_SMD:R_0805_2012Metric_Pad1.20x1.40mm_HandSolder, F.Cu at (209.9, 70.0)
- added RV14: P4_C, Potentiometer_THT:Potentiometer_Bourns_PTV09A-1_Single_Vertical, F.Cu at (108.5, 121.4)
- added RV15: P5_C, Potentiometer_THT:Potentiometer_Bourns_PTV09A-1_Single_Vertical, F.Cu at (108.5, 152.4)
- added RV16: P1_D, Potentiometer_THT:Potentiometer_Bourns_PTV09A-1_Single_Vertical, F.Cu at (134.5, 37.4)
- added RV17: P2_D, Potentiometer_THT:Potentiometer_Bourns_PTV09A-1_Single_Vertical, F.Cu at (134.5, 65.4)
- added RV18: P3_D, Potentiometer_THT:Potentiometer_Bourns_PTV09A-1_Single_Vertical, F.Cu at (134.5, 93.4)
- added RV19: P4_D, Potentiometer_THT:Potentiometer_Bourns_PTV09A-1_Single_Vertical, F.Cu at (134.5, 121.4)
- added RV20: P5_D, Potentiometer_THT:Potentiometer_Bourns_PTV09A-1_Single_Vertical, F.Cu at (134.5, 152.4)
- added RV21: P1_G, Potentiometer_THT:Potentiometer_Bourns_PTV09A-1_Single_Vertical, F.Cu at (193.8, 92.7)
- added RV22: P2_G, Potentiometer_THT:Potentiometer_Bourns_PTV09A-1_Single_Vertical, F.Cu at (193.8, 107.4)
- added RV23: P3_G, Potentiometer_THT:Potentiometer_Bourns_PTV09A-1_Single_Vertical, F.Cu at (193.8, 122.2)
- added U2: TCA9548APWR, Package_SO:TSSOP-24_4.4x7.8mm_P0.65mm, F.Cu at (212.3, 57.9)
- added U3: MAX11616, Package_SO:QSOP-16_3.9x4.9mm_P0.635mm, F.Cu at (212.2, 74.7)
- C1: value 1uF -> 10uF; footprint Capacitor_SMD:C_1206_3216Metric_Pad1.33x1.80mm_HandSolder -> Capacitor_SMD:C_0805_2012Metric_Pad1.18x1.45mm_HandSolder
- C2: footprint Capacitor_SMD:C_1206_3216Metric_Pad1.33x1.80mm_HandSolder -> Capacitor_SMD:C_0603_1608Metric_Pad1.08x0.95mm_HandSolder
- J1: value MPLEX-IN -> IN; footprint Connector_PinHeader_2.54mm:PinHeader_1x04_P2.54mm_Vertical -> Connector_JST:JST_PH_S4B-PH-K_1x04_P2.00mm_Horizontal
- R1, R2: footprint Resistor_SMD:R_1206_3216Metric_Pad1.30x1.75mm_HandSolder -> Resistor_SMD:R_0805_2012Metric_Pad1.20x1.40mm_HandSolder
- RV1: value L1_Pot -> P1_A; footprint eqLibrary:Potentiometer_Bourns_PTV09A-1_Single_Vertical -> Potentiometer_THT:Potentiometer_Bourns_PTV09A-1_Single_Vertical
- RV10: value R2_Pot -> P5_B; footprint eqLibrary:Potentiometer_Bourns_PTV09A-1_Single_Vertical -> Potentiometer_THT:Potentiometer_Bourns_PTV09A-1_Single_Vertical
- RV11: value R3_Pot -> P1_C; footprint eqLibrary:Potentiometer_Bourns_PTV09A-1_Single_Vertical -> Potentiometer_THT:Potentiometer_Bourns_PTV09A-1_Single_Vertical
- RV12: value R4_Pot -> P2_C; footprint eqLibrary:Potentiometer_Bourns_PTV09A-1_Single_Vertical -> Potentiometer_THT:Potentiometer_Bourns_PTV09A-1_Single_Vertical
- RV13: value R5_Pot -> P3_C; footprint eqLibrary:Potentiometer_Bourns_PTV09A-1_Single_Vertical -> Potentiometer_THT:Potentiometer_Bourns_PTV09A-1_Single_Vertical
- RV2: value L2_Pot -> P2_A; footprint eqLibrary:Potentiometer_Bourns_PTV09A-1_Single_Vertical -> Potentiometer_THT:Potentiometer_Bourns_PTV09A-1_Single_Vertical
- RV3: value L3_Pot -> P3_A; footprint eqLibrary:Potentiometer_Bourns_PTV09A-1_Single_Vertical -> Potentiometer_THT:Potentiometer_Bourns_PTV09A-1_Single_Vertical
- RV4: value L4_Pot -> P4_A; footprint eqLibrary:Potentiometer_Bourns_PTV09A-1_Single_Vertical -> Potentiometer_THT:Potentiometer_Bourns_PTV09A-1_Single_Vertical
- RV5: value L5_Pot -> P5_A; footprint eqLibrary:Potentiometer_Bourns_PTV09A-1_Single_Vertical -> Potentiometer_THT:Potentiometer_Bourns_PTV09A-1_Single_Vertical
- RV6: value C1_Pot -> P1_B; footprint eqLibrary:Potentiometer_Bourns_PTV09A-1_Single_Vertical -> Potentiometer_THT:Potentiometer_Bourns_PTV09A-1_Single_Vertical
- RV7: value C2_Pot -> P2_B; footprint eqLibrary:Potentiometer_Bourns_PTV09A-1_Single_Vertical -> Potentiometer_THT:Potentiometer_Bourns_PTV09A-1_Single_Vertical
- RV8: value C3_Pot -> P3_B; footprint eqLibrary:Potentiometer_Bourns_PTV09A-1_Single_Vertical -> Potentiometer_THT:Potentiometer_Bourns_PTV09A-1_Single_Vertical
- RV9: value R1_Pot -> P4_B; footprint eqLibrary:Potentiometer_Bourns_PTV09A-1_Single_Vertical -> Potentiometer_THT:Potentiometer_Bourns_PTV09A-1_Single_Vertical
- U1: value CD74HC4067M -> MAX11616; footprint Package_SO:SOIC-24W_7.5x15.4mm_P1.27mm -> Package_SO:QSOP-16_3.9x4.9mm_P0.635mm
- moved H2 145.6 mm to (52.0, 32.5), turned to 90 degrees
- moved RV1 129.0 mm to (56.5, 37.4), turned to -90 degrees
- moved H4 124.8 mm to (144.0, 32.5), turned to 90 degrees
- moved H1 120.5 mm to (52.0, 174.5), turned to 90 degrees
- moved RV6 118.9 mm to (82.5, 37.4), turned to -90 degrees
- moved RV11 101.6 mm to (108.5, 37.4), turned to -90 degrees
- moved RV9 100.8 mm to (82.5, 121.4), turned to -90 degrees
- moved RV2 97.5 mm to (56.5, 65.4), turned to -90 degrees
- moved H3 94.4 mm to (144.0, 174.5), turned to 90 degrees
- moved RV5 85.1 mm to (56.5, 152.4), turned to -90 degrees
- moved J1 83.3 mm to (170.5, 33.5), turned to 90 degrees
- moved RV3 74.2 mm to (56.5, 93.4), turned to -90 degrees
- moved RV10 73.0 mm to (82.5, 152.4), turned to -90 degrees
- moved RV12 72.8 mm to (108.5, 65.4), turned to -90 degrees
- moved U1 69.6 mm to (96.5, 69.0), turned to 0 degrees
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Connections:
- C1 pad 1: /SW1 -> Net-(U1-Vdd)
- C2 pad 1: /SW2 -> Net-(U1-Vdd)
- J1 pad 1: /MPLEX-S0 -> GND
- J1 pad 2: /MPLEX-S1 -> +5V
- J1 pad 3: /MPLEX-S2 -> /SDA
- J1 pad 4: /MPLEX-S3 -> /SCL
- R1 pad 2: /SW1 -> /SDA
- R2 pad 2: /SW2 -> /SCL
- RV1 pad 2: /POT-L1 -> /A0
- RV10 pad 2: /POT-R2 -> /A9
- RV11 pad 2: /POT-R3 -> /AA0
- RV12 pad 2: /POT-R4 -> /AA1
- RV13 pad 2: /POT-R5 -> /AA2
- RV2 pad 2: /POT-L2 -> /A1
- RV3 pad 2: /POT-L3 -> /A2
- RV4 pad 2: /POT-L4 -> /A3
- RV5 pad 2: /POT-L5 -> /A4
- RV6 pad 2: /POT-C1 -> /A5
- RV7 pad 2: /POT-C2 -> /A6
- RV8 pad 2: /POT-C3 -> /A7
- RV9 pad 2: /POT-R1 -> /A8
- U1 pad 1: /MPLEX-AP -> /A11
- U1 pad 10: /MPLEX-S0 -> /A5
- U1 pad 11: /MPLEX-S1 -> /A6
- U1 pad 12: GND -> /A7
- U1 pad 13: /MPLEX-S3 -> /SC0
- U1 pad 14: /MPLEX-S2 -> /SD0
- U1 pad 16: /POT-R1 -> Net-(U1-Vdd)
- U1 pad 2: /POT-C3 -> /A10
- U1 pad 3: /POT-C2 -> /A9
- U1 pad 4: /POT-L5 -> /A8
- U1 pad 5: /POT-L4 -> /A0
- U1 pad 6: /POT-L3 -> /A1
- U1 pad 7: /POT-L2 -> /A2
- U1 pad 8: /POT-L1 -> /A3
- U1 pad 9: /POT-C1 -> /A4
Routing:
- net +5V: track 564.0 -> 0.00 mm, vias 4 -> 0
- net GND: track 342.8 -> 0.00 mm, vias 26 -> 0
- net /MPLEX-S0: track 237.9 -> 0.00 mm
- net /MPLEX-S1: track 231.2 -> 0.00 mm
- net /MPLEX-S2: track 218.5 -> 0.00 mm
- net /MPLEX-S3: track 208.6 -> 0.00 mm
- net /SW1: track 160.1 -> 0.00 mm
- net /POT-R5: track 120.4 -> 0.00 mm
- net /POT-L5: track 116.3 -> 0.00 mm
- net /SW2: track 98.1 -> 0.00 mm
- net /POT-R4: track 85.8 -> 0.00 mm
- net /POT-L4: track 81.7 -> 0.00 mm
- net /POT-C3: track 67.0 -> 0.00 mm
- net /POT-R3: track 59.5 -> 0.00 mm
- net /POT-L3: track 55.8 -> 0.00 mm
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Other:
- board size 150 x 100 mm -> 100 x 150 mm
