File: KiCAD/0x1F/EquBoard/EquBoard.kicad_sch (KiCad schematic)
At the start: 30 parts, among them J1 MPLEX-IN, J2 MPLEX-OUT, J3 MPLEX-AP, J4 LED-CONN, SW1 SW_LED_1, SW2 SW_LED_2, U1 CD74HC4067M

Commit message: pre firm
Parts:
- removed J2: MPLEX-OUT, Connector_PinHeader_2.54mm:PinHeader_1x04_P2.54mm_Vertical, symbol Connector_Generic:Conn_01x04
- removed J3: MPLEX-AP, Connector_PinHeader_2.54mm:PinHeader_1x03_P2.54mm_Vertical, symbol Connector_Generic:Conn_01x03
- removed J4: LED-CONN, Connector_PinHeader_2.54mm:PinHeader_1x02_P2.54mm_Vertical, symbol Connector_Generic:Conn_01x02
- removed U1: CD74HC4067M, Package_SO:SOIC-24W_7.5x15.4mm_P1.27mm, symbol 74xx:CD74HC4067M
- added C3: 10uF, Capacitor_SMD:C_0805_2012Metric_Pad1.18x1.45mm_HandSolder, symbol Device:C_Small
- added C4: 1uF, Capacitor_SMD:C_0603_1608Metric_Pad1.08x0.95mm_HandSolder, symbol Device:C_Small
- added C5: 100nF, Capacitor_SMD:C_0603_1608Metric_Pad1.08x0.95mm_HandSolder, symbol Device:C_Small
- added JP1: A0, Jumper:SolderJumper-2_P1.3mm_Open_RoundedPad1.0x1.5mm, symbol Jumper:SolderJumper_2_Open
- added JP2: A1, Jumper:SolderJumper-2_P1.3mm_Open_RoundedPad1.0x1.5mm, symbol Jumper:SolderJumper_2_Open
- added R3: 5R, Resistor_SMD:R_0805_2012Metric_Pad1.20x1.40mm_HandSolder, symbol Device:R_Small
- added R4, R5, R6, R7: 10K, Resistor_SMD:R_0805_2012Metric_Pad1.20x1.40mm_HandSolder, symbol Device:R_Small
- added U2: ADS7830, Package_SO:TSSOP-16_4.4x5mm_P0.65mm, symbol Analog_DAC:ADS7830
- J1: value MPLEX-IN -> IN; footprint Connector_PinHeader_2.54mm:PinHeader_1x04_P2.54mm_Vertical -> Connector_JST:JST_PH_S4B-PH-K_1x04_P2.00mm_Horizontal
Connections:
- net MPLEX-S0 is gone; now on net GND: J1.1 (Pin_1)
- net MPLEX-S1 is gone; now on net +5V: J1.2 (Pin_2)
- net +5V: now also R3.1, R6.1, R7.1
- net GND: now also C3.2, C4.2, C5.2, R4.2, R5.2, U2.9 (GND)
- net MPLEX-S2 renamed SDA
- net SDA: now also R6.2, U2.15 (SDA)
- net MPLEX-S3 renamed SCL
- net SCL: now also R7.2, U2.14 (SCL)
- new net: JP2.2 (B), R5.1
- new net: C3.1, C4.1, C5.1, R3.2, U2.10 (REFin/REFout), U2.16 (VDD)
- new net: JP1.2 (B), R4.1
- new net A0: JP1.1 (A), U2.12 (A0)
- new net A1: JP2.1 (A), U2.13 (A1)
- new net POT1: U2.1 (CH0)
- new net POT2: U2.3 (CH2)
- new net POT3: U2.5 (CH4)
- new net POT4: U2.7 (CH6)
- new net POT5: U2.2 (CH1)
- new net POT6: U2.4 (CH3)
- new net POT7: U2.6 (CH5)
- new net POT8: U2.8 (CH7)

Commit message: rp2040 zero
Parts:
- removed C1, C2: 1uF, Capacitor_SMD:C_1206_3216Metric_Pad1.33x1.80mm_HandSolder, symbol Device:C_Small
- removed JP1: A0, Jumper:SolderJumper-2_P1.3mm_Open_RoundedPad1.0x1.5mm, symbol Jumper:SolderJumper_2_Open
- removed JP2: A1, Jumper:SolderJumper-2_P1.3mm_Open_RoundedPad1.0x1.5mm, symbol Jumper:SolderJumper_2_Open
- removed R1, R2: 10K, Resistor_SMD:R_1206_3216Metric_Pad1.30x1.75mm_HandSolder, symbol Device:R_Small
- removed R4: 10K, Resistor_SMD:R_0805_2012Metric_Pad1.20x1.40mm_HandSolder, symbol Device:R_Small
- removed SW1: SW_LED_1, eqLibrary:led switch, symbol Switch:SW_Push_LED
- removed SW2: SW_LED_2, eqLibrary:led switch, symbol Switch:SW_Push_LED
- removed U2: ADS7830, Package_SO:TSSOP-16_4.4x5mm_P0.65mm, symbol Analog_DAC:ADS7830
- added C4: 10uF, Capacitor_SMD:C_0805_2012Metric_Pad1.18x1.45mm_HandSolder, symbol Device:C_Small
- added C5: 1uF, Capacitor_SMD:C_0603_1608Metric_Pad1.08x0.95mm_HandSolder, symbol Device:C_Small
- added R5: 5R, Resistor_SMD:R_0805_2012Metric_Pad1.20x1.40mm_HandSolder, symbol Device:R_Small
- added RV14: P4_C, Potentiometer_THT:Potentiometer_Bourns_PTV09A-1_Single_Vertical, symbol Device:R_Potentiometer_Small
- added RV15: P5_C, Potentiometer_THT:Potentiometer_Bourns_PTV09A-1_Single_Vertical, symbol Device:R_Potentiometer_Small
- added RV16: P1_D, Potentiometer_THT:Potentiometer_Bourns_PTV09A-1_Single_Vertical, symbol Device:R_Potentiometer_Small
- added RV17: P2_D, Potentiometer_THT:Potentiometer_Bourns_PTV09A-1_Single_Vertical, symbol Device:R_Potentiometer_Small
- added RV18: P3_D, Potentiometer_THT:Potentiometer_Bourns_PTV09A-1_Single_Vertical, symbol Device:R_Potentiometer_Small
- added RV19: P4_D, Potentiometer_THT:Potentiometer_Bourns_PTV09A-1_Single_Vertical, symbol Device:R_Potentiometer_Small
- added RV20: P5_D, Potentiometer_THT:Potentiometer_Bourns_PTV09A-1_Single_Vertical, symbol Device:R_Potentiometer_Small
- added RV6: P1_B, Potentiometer_THT:Potentiometer_Bourns_PTV09A-1_Single_Vertical, symbol Device:R_Potentiometer_Small
- added RV7: P2_B, Potentiometer_THT:Potentiometer_Bourns_PTV09A-1_Single_Vertical, symbol Device:R_Potentiometer_Small
- added RV8: P3_B, Potentiometer_THT:Potentiometer_Bourns_PTV09A-1_Single_Vertical, symbol Device:R_Potentiometer_Small
- added U1, U3: MAX11616, Package_SO:QSOP-16_3.9x4.9mm_P0.635mm, symbol Analog_ADC:MAX11616
- added U2: TCA9548APWR, Package_SO:TSSOP-24_4.4x7.8mm_P0.65mm, symbol Interface_Expansion:TCA9548APWR
- C3: renamed from C5; value 100nF -> 10uF
- RV1: value L1_Pot -> P1_A
- RV10: value R2_Pot -> P5_B
- RV11: value R3_Pot -> P1_C
- RV12: value R4_Pot -> P2_C
- RV13: value R5_Pot -> P3_C
- RV2: value L2_Pot -> P2_A
- RV21: renamed from RV6; value C1_Pot -> P1_G
- RV22: renamed from RV7; value C2_Pot -> P2_G
- RV23: renamed from RV8; value C3_Pot -> P3_G
- RV3: value L3_Pot -> P3_A
- RV4: value L4_Pot -> P4_A
- RV5: value L5_Pot -> P5_A
- RV9: value R1_Pot -> P4_B
- renumbered C3 to C1, C4 to C2, R6 to R1, R7 to R2, R5 to R4
Connections:
- net POT-L1 is gone; now on net A0: RV1.2
- net POT-L2 is gone; now on net A1: RV2.2
- net +5V: now also C3.1, R4.1, R5.1, RV14.1, RV15.1, RV16.1, RV17.1, RV18.1, RV19.1, RV20.1, RV6.1, RV7.1, RV8.1, U2.1 (A0), U2.2 (A1), U2.21 (A2), U2.24 (VCC)
- net A0: now also U1.5 (AIN0)
- net A1: now also U1.6 (AIN1)
- net GND: now also C4.2, C5.2, RV14.3, RV15.3, RV16.3, RV17.3, RV18.3, RV19.3, RV20.3, RV6.3, RV7.3, RV8.3, U1.15 (GND), U2.12 (GND), U3.15 (GND); no longer R4.2
- net SCL: now also U2.22 (SCL)
- net SDA: now also U2.23 (SDA)
- net at C1.1, C2.1, R3.2: now also U1.16 (Vdd); no longer C3.1
- net POT-C1 renamed A10
- net A10: now also U1.2 (AIN10)
- net POT-C2 renamed A11
- net A11: now also U1.1 (AIN11)
- net POT-C3 renamed AA10
- net AA10: now also U3.2 (AIN10)
- net POT-L3 renamed A2
- net A2: now also U1.7 (AIN2)
- net POT-L4 renamed A3
- net A3: now also U1.8 (AIN3)
- net POT-L5 renamed A4
- net A4: now also U1.9 (AIN4)
- net POT-R1 renamed A8
- net A8: now also U1.4 (AIN8)
- net POT-R2 renamed A9
- net A9: now also U1.3 (AIN9)
- net POT-R3 renamed AA0
- net AA0: now also U3.5 (AIN0)
- net POT-R4 renamed AA1
- net AA1: now also U3.6 (AIN1)
- net POT-R5 renamed AA2
- net AA2: now also U3.7 (AIN2)
- new net: R4.2, U2.3 (~{RESET})
- new net: C4.1, C5.1, R5.2, U3.16 (Vdd)
- new net A5: RV6.2, U1.10 (AIN5)
- new net A6: RV7.2, U1.11 (AIN6)
- new net A7: RV8.2, U1.12 (AIN7)
- new net AA3: RV14.2, U3.8 (AIN3)
- new net AA4: RV15.2, U3.9 (AIN4)
- new net AA5: RV16.2, U3.10 (AIN5)
- new net AA6: RV17.2, U3.11 (AIN6)
- new net AA7: RV18.2, U3.12 (AIN7)
- new net AA8: RV19.2, U3.4 (AIN8)
- new net AA9: RV20.2, U3.3 (AIN9)
- new net SC0: U1.13 (SCL), U2.5 (SC0)
- new net SC1: U2.7 (SC1), U3.13 (SCL)
- new net SD0: U1.14 (SDA), U2.4 (SD0)
- new net SD1: U2.6 (SD1), U3.14 (SDA)
- no-connect marks 1 -> 13
Other:
- moved on the sheet: C1, C2, C3, H1, H2, H3, H4, H5, H6, J1, R1, R2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
